File: Hardware/RF_Transceiver.sch (KiCad schematic (older format))
At the start: 36 parts, among them P1 GND, P10 Vin, P11 GND, P12 GND, P2 RESET, P3 ~CSCON, P4 IRQ0, P5 SDI, P6 SCK, P7 SDO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

Commit message: Complete and abandonned
Parts:
- FL1: value TA0801A -> SF2314E
Changed lines of the file:
@@
 encoding utf-8
 Sheet 1 1
-Title ""
-Date ""
-Rev ""
-Comp ""
-Comment1 ""
-Comment2 ""
+Title "RF Transceiver"
+Date "2019-04-19"
+Rev "00"
+Comp "EsseivaN"
+Comment1 "Author : Esseiva Nicolas"
+Comment2 "RF, 868MHz, Transceiver (TxRx) using MRF89XA"
 Comment3 ""
 Comment4 ""
@@
 P 3250 1500
 F 0 "FL1" H 3400 1965 50  0000 C CNN
-F 1 "TA0801A" H 3400 1874 50  0000 C CNN
+F 1 "SF2314E" H 3400 1874 50  0000 C CNN
 F 2 "" H 3250 1500 50  0001 C CNN
 F 3 "" H 3250 1500 50  0001 C CNN
